Commit message: exercice_5_b_suite
suite de l'exercice 5b

File: src/gpg_remote/gpg_remote/config/gopigo3.urdf (robot description, URDF)
Before this commit: robot gopigo3, 0 links, 0 joints
Links:
- added link base_link, mass 0.1; collision cylinder length=0.005 radius=0.075; visual cylinder length=0.005 radius=0.075
- added link camera_link, mass 0.001; collision box size=0.01 0.01 0.01; visual box size=0.01 0.01 0.01
- added link left_wheel_link, mass 0.001; collision cylinder length=0.04 radius=0.0375; visual cylinder length=0.04 radius=0.0375
- added link right_wheel_link, mass 0.001; collision cylinder length=0.04 radius=0.0375; visual cylinder length=0.04 radius=0.0375
- added link robot_support_link, mass 0.1; collision cylinder length=01875 radius=0.01; visual cylinder length=0.01875 radius=0.01
- added link servo_link, mass 0.001; collision box size=0.03 0.03 0.03; visual box size=0.03 0.03 0.03
Joints:
- added joint camera_to_servo_link: type fixed, parent servo_link, child camera_link, origin xyz=0.015 0 0 rpy=-1.57 0 0
- added joint left_wheel: type continuous, parent base_link, child left_wheel_link, origin xyz=0 0.062 0.0375 rpy=0 0 0, axis 0 1 0
- added joint right_wheel: type continuous, parent base_link, child right_wheel_link, origin xyz=0 -0.062 0.0375 rpy=0 0 0, axis 0 1 0
- added joint robot_support_joint: type continuous, parent base_link, child robot_support_link, origin xyz=-0.065 0 0.0375 rpy=0 0 0, axis 0 0 1
- added joint servo: type revolute, parent base_link, child servo_link, origin xyz=0.075 0 0.065 rpy=0 0 0, axis 0 0 1, limit lower=-1.57 upper=1.57 effort=1 velocity=1
